Commit message: feat(vision): integrate Shi-Tomasi feature tracking and dynamic camera/lidar bridging

File: src/swarm_core/urdf/drone.urdf.xacro (robot description, xacro)
@@ -1,4 +1,5 @@
 <?xml version="1.0"?>
 <robot name="swarm_drone" xmlns:xacro="http://ros.org/wiki/xacro">
+  <xacro:arg name="drone_name" default="alpha"/>
   <xacro:property name="base_mass" value="0.5"/>
   <xacro:property name="base_radius" value="0.1"/>
@@ -33,4 +34,10 @@
     <origin xyz="0.1 0 0" rpy="0 0 0"/>
   </joint>
+  <link name="lidar_link"/>
+  <joint name="lidar_joint" type="fixed">
+    <parent link="base_link"/>
+    <child link="lidar_link"/>
+    <origin xyz="0 0 0.05" rpy="0 0 0"/>
+  </joint>
   <gazebo reference="camera_link">
     <sensor name="front_camera" type="camera">
@@ -43,5 +50,19 @@
       <update_rate>30</update_rate>
       <visualize>true</visualize>
-      <topic>camera/image_raw</topic>
+      <topic>/$(arg drone_name)/camera/image_raw</topic>
+    </sensor>
+  </gazebo>
+  <gazebo reference="lidar_link">
+    <sensor name="lidar_sensor" type="gpu_lidar">
+      <always_on>1</always_on>
+      <update_rate>10</update_rate>
+      <visualize>true</visualize>
+      <topic>/$(arg drone_name)/scan</topic>
+      <ray>
+        <scan>
+          <horizontal><samples>360</samples><resolution>1</resolution><min_angle>-3.14159</min_angle><max_angle>3.14159</max_angle></horizontal>
+        </scan>
+        <range><min>0.2</min><max>10.0</max><resolution>0.01</resolution></range>
+      </ray>
     </sensor>
   </gazebo>
